Commit message: Add a functional lifting unit

File: urdf/elevator/elevator.urdf.xacro (robot description, xacro)
@@ -2,5 +2,5 @@
 <robot xmlns:xacro="http://www.ros.org/wiki/xacro">
 	<xacro:include filename="$(find rb1_ros2_description)/urdf/elevator/elevator.gazebo.xacro"/>
-	<xacro:macro name="elevator_platform" params="prefix parent hq *origin">
+	<xacro:macro name="elevator_platform" params="prefix parent hq">
 	<!-- PARAMS: -->
 	<!-- name : name of the link: -->
@@ -9,6 +9,5 @@
 		<inertia  ixx="${(m*(h*h+d*d))/12}" ixy = "0" ixz = "0"
               iyy="${(m*(w*w+d*d))/12}" iyz = "0"
-              izz="${(m*(w*w+h*h))/12}"
-     />
+              izz="${(m*(w*w+h*h))/12}"/>
     </xacro:macro>
 	<!-- ELEVATOR_BASE_LINK -->
@@ -16,5 +15,6 @@
 		<parent link="${parent}"/>
 		<child link="${prefix}_base_link"/>
-		<xacro:insert_block name="origin" />
+        <origin xyz="0 0 0.23" rpy="0 0 0"/>
+		<!--xacro:insert_block name="origin" /-->
 	</joint>
 	<link name="${prefix}_base_link">
@@ -29,5 +29,5 @@
 			<mass value="0.005" />
 			<origin xyz="0 0 -0.27" />
-			<solid_cuboid_inertia m="0.005" h="0.05" d="0.05" w="0.05"/>
+			<xacro:solid_cuboid_inertia m="0.005" h="0.05" d="0.05" w="0.05"/>
 		</inertial>
 		<visual>
@@ -71,5 +71,5 @@
 			<mass value="0.005" />
 			<origin xyz="0 0 -0.27" />
-			<solid_cuboid_inertia m="0.005" h="0.05" d="0.05" w="0.05"/>
+			<xacro:solid_cuboid_inertia m="0.005" h="0.05" d="0.05" w="0.05"/>
 		</inertial>
 		<visual>

File: urdf/ueye_cp_gige.urdf.xacro (robot description, xacro)
@@ -3,5 +3,5 @@
   <xacro:macro name="sensor_ueye_cp_gige" params="prefix parent *origin">
     <joint name="${prefix}_joint" type="fixed">
-      <insert_block name="origin"/>
+      <xacro:insert_block name="origin"/>
       <parent link="${parent}"/>
       <child link="${prefix}_base_link"/>

File: xacro/rb1_ros2_base.urdf.xacro (robot description, xacro)
@@ -76,5 +76,45 @@
 		<origin xyz="0.234 0.0 0.092" rpy="0 0 0"/>
 	</xacro:sensor_orbbec_astra>
-	<!-- Gazebo ros2 control plugins -->
-	<!-- <xacro:ros2_control/> -->
+    <!-- ELEVATOR -->
+    <xacro:elevator_platform prefix="$(arg prefix)elevator" parent="$(arg prefix)base_link" hq="${hq}" />
+    <!-- <xacro:ros2_control/> -->
+    <ros2_control name="diffdrive" type="system">
+      <hardware>
+          <plugin>gazebo_ros2_control/GazeboSystem</plugin>
+      </hardware>
+      <joint name="robot_left_wheel_joint">
+        <command_interface name="velocity">
+          <param name="min">-1</param>
+          <param name="max">1</param>
+        </command_interface>
+        <state_interface name="position"/>
+        <state_interface name="velocity"/>
+        <state_interface name="effort"/>
+      </joint>
+      <joint name="robot_right_wheel_joint">
+        <command_interface name="velocity">
+          <param name="min">-1</param>
+          <param name="max">1</param>
+        </command_interface>
+        <state_interface name="position"/>
+        <state_interface name="velocity"/>
+        <state_interface name="effort"/>
+      </joint>
+        <joint name="robot_elevator_platform_joint">
+        <command_interface name="effort" >
+            <param name="min">-1</param>
+            <param name="max">1</param>
+        </command_interface>
+        <state_interface name="position"/>
+        <state_interface name="velocity"/>
+        <state_interface name="effort"/>
+      </joint>
+    </ros2_control>
+    <!-- Gazebo ros2 control plugins -->
+    <gazebo>
+        <plugin name="gazebo_ros2_control" filename="libgazebo_ros2_control.so">
+            <robot_sim_type>gazebo_ros2_control/GazeboSystem</robot_sim_type>
+            <parameters>$(find rb1_ros2_description)/config/rb1_controller.yaml</parameters>
+        </plugin>
+    </gazebo>
 </robot>
